File: frambuesa-rev-a/frambuesa-rev-a.kicad_sch (KiCad schematic)
At the start: 38 parts, among them J3 Conn_02x18_Odd_Even, J4 Conn_02x18_Odd_Even, J5 USB_C_Receptacle_USB2.0_16P, SW1 PTS 636, U1 RP2040, U2 AMS1117-5.0, U3 W25Q128JVS, Y1 Crystal_GND24

Commit message: agregar bibliotecas
Parts:
- C12, C18: footprint (none) -> frambuesa-rev-a:C1206
- C13, C19, C20: footprint (none) -> frambuesa-rev-a:C0402
- J5: footprint (none) -> frambuesa-rev-a:USB-C_SMD-TYPE-C-31-M-12_1
- R4, R6, R7: footprint (none) -> frambuesa-rev-a:R0402
- SW1: footprint (none) -> frambuesa-rev-a:KEY-SMD_L6.0-W3.5-LS8.7
- U3: footprint Package_SO:SOIC-8_5.3x5.3mm_P1.27mm -> frambuesa-rev-a:SOIC-8_L5.3-W5.3-P1.27-LS8.0-BL
Changed lines of the file:
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@@
 			)
 		)
-		(property "Footprint" "Package_SO:SOIC-8_5.3x5.3mm_P1.27mm"
+		(property "Footprint" "frambuesa-rev-a:SOIC-8_L5.3-W5.3-P1.27-LS8.0-BL"
 			(at 69.85 288.29 0)
 			(hide yes)
@@
 			)
 		)
-		(property "Footprint" ""
+		(property "Footprint" "frambuesa-rev-a:R0402"
 			(at 84.582 239.395 90)
 			(hide yes)
@@
 			)
 		)
-		(property "Footprint" ""
+		(property "Footprint" "frambuesa-rev-a:R0402"
 			(at 75.057 239.395 90)
 			(hide yes)
@@
 			)
 		)
-		(property "Footprint" ""
+		(property "Footprint" "frambuesa-rev-a:C0402"
 			(at 175.5902 236.855 0)
 			(hide yes)
@@
 			)
 		)
-		(property "Footprint" ""
+		(property "Footprint" "frambuesa-rev-a:C1206"
 			(at 160.3502 236.855 0)
 			(hide yes)
@@
 			)
 		)
-		(property "Footprint" ""
+		(property "Footprint" "frambuesa-rev-a:C0402"
 			(at 82.2452 290.83 0)
 			(hide yes)
@@
 			)
 		)
-		(property "Footprint" ""
+		(property "Footprint" "frambuesa-rev-a:USB-C_SMD-TYPE-C-31-M-12_1"
 			(at 36.83 241.3 0)
 			(hide yes)
@@
 			)
 		)
-		(property "Footprint" ""
+		(property "Footprint" "frambuesa-rev-a:KEY-SMD_L6.0-W3.5-LS8.7"
 			(at 27.94 303.53 0)
 			(hide yes)
@@
 			)
 		)
-		(property "Footprint" ""
+		(property "Footprint" "frambuesa-rev-a:C1206"
 			(at 107.6452 237.49 0)
 			(hide yes)
@@
 			)
 		)
-		(property "Footprint" ""
+		(property "Footprint" "frambuesa-rev-a:C0402"
 			(at 122.8852 237.49 0)
 			(hide yes)
@@
 			)
 		)
-		(property "Footprint" ""
+		(property "Footprint" "frambuesa-rev-a:R0402"
 			(at 49.022 290.195 90)
 			(hide yes)
