File: frambu-v-0-rev-a/frambu-v-0-rev-a.kicad_sch (KiCad schematic)
At the start: 38 parts, among them J3 Conn_02x18_Odd_Even, J4 Conn_02x18_Odd_Even, J5 USB_C_Receptacle_USB2.0_16P, SW1 PTS 636, U1 RP2040, U2 AMS1117-5.0, U3 W25Q128JVS, Y1 Crystal_GND24

Commit message: nombre nuevo frambu
Parts:
- C12, C18: footprint frambuesa-rev-a:C1206 -> frambu-v-0-rev-a:C1206
- C13, C19, C20: footprint frambuesa-rev-a:C0402 -> frambu-v-0-rev-a:C0402
- J5: footprint frambuesa-rev-a:USB-C_SMD-TYPE-C-31-M-12_1 -> frambu-v-0-rev-a:USB-C_SMD-TYPE-C-31-M-12_1
- R4, R6, R7: footprint frambuesa-rev-a:R0402 -> frambu-v-0-rev-a:R0402
- SW1: footprint frambuesa-rev-a:KEY-SMD_L6.0-W3.5-LS8.7 -> frambu-v-0-rev-a:KEY-SMD_L6.0-W3.5-LS8.7
- U3: footprint frambuesa-rev-a:SOIC-8_L5.3-W5.3-P1.27-LS8.0-BL -> frambu-v-0-rev-a:SOIC-8_L5.3-W5.3-P1.27-LS8.0-BL
Other:
- title: frambuesa -> frambu

Commit message: agregar sgtl500
Parts:
- removed H3, H4: MountingHole, MountingHole:MountingHole_3.2mm_M3, symbol Mechanical:MountingHole
- added U4: SGTL5000XNLA3, Package_DFN_QFN:QFN-20-1EP_3x3mm_P0.4mm_EP1.65x1.65mm, symbol Audio:SGTL5000XNLA3
Other:
- note removed: "flash FP pending"
- note removed: "poder FP pending"
- note removed: "usb FP pending"
Changed lines of the file:
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@@
 	(title_block
 		(title "frambu")
-		(date "2026-09-17")
+		(date "2026-10-03")
 		(rev "rev-a")
 		(company "piruetas SpA")
 	)
-	(text "flash FP pending"
-		(exclude_from_sim no)
-		(at 30.988 288.29 0)
-		(effects
-			(font
-				(size 1.27 1.27)
-			)
-		)
-	)
-	(text "usb FP pending\n\n"
-		(exclude_from_sim no)
-		(at 60.452 217.678 0)
-		(effects
-			(font
-				(size 1.27 1.27)
-			)
-		)
-	)
 	(text "entradas y salidas\n"
 		(exclude_from_sim no)
@@
 		)
 	)
-	(text "poder FP pending\n"
-		(exclude_from_sim no)
-		(at 140.335 215.265 0)
-		(effects
-			(font
-				(size 1.27 1.27)
-			)
-		)
-	)
 	(text "cristal TODO\n\n "
 		(exclude_from_sim no)
@@
 	)
 	(symbol
-		(lib_id "Mechanical:MountingHole")
-		(at 229.87 367.03 0)
-		(unit 1)
-		(body_style 1)
-		(exclude_from_sim no)
-		(in_bom no)
-		(on_board yes)
-		(in_pos_files yes)
-		(dnp no)
-		(fields_autoplaced yes)
-		(property "Reference" "H4"
-			(at 232.41 365.7599 0)
-			(show_name no)
-			(do_not_autoplace no)
-			(effects
-				(font
-					(size 1.27 1.27)
-				)
-				(justify left)
-			)
-		)
-		(property "Value" "MountingHole"
-			(at 232.41 368.2999 0)
-			(show_name no)
-			(do_not_autoplace no)
-			(effects
-				(font
-					(size 1.27 1.27)
-				)
-				(justify left)
-			)
-		)
-		(property "Footprint" "MountingHole:MountingHole_3.2mm_M3"
-			(at 229.87 367.03 0)
-			(hide yes)
-			(show_name no)
-			(do_not_autoplace no)
-			(effects
-				(font
-					(size 1.27 1.27)
-				)
-			)
-		)
-		(property "Datasheet" ""
-			(at 229.87 367.03 0)
-			(hide yes)
-			(show_name no)
-			(do_not_autoplace no)
-			(effects
-				(font
-					(size 1.27 1.27)
-				)
-			)
-		)
-		(property "Description" "Mounting Hole without connection"
-			(at 229.87 367.03 0)
-			(hide yes)
-			(show_name no)
-			(do_not_autoplace no)
-			(effects
-				(font
-					(size 1.27 1.27)
-				)
-			)
-		)
-		(instances
-			(project "frambu-v-0-rev-a"
-				(path "/abe203a7-9d57-48b6-8b01-f2c6245f8096"
-					(reference "H4")
-					(unit 1)
-				)
-			)
-		)
-	)
-	(symbol
 		(lib_id "Device:R")
 		(at 97.79 123.19 90)
@@
 	)
 	(symbol
-		(lib_id "Mechanical:MountingHole")
-		(at 229.87 360.68 0)
-		(unit 1)
-		(body_style 1)
-		(exclude_from_sim no)
-		(in_bom no)
-		(on_board yes)
-		(in_pos_files yes)
-		(dnp no)
-		(fields_autoplaced yes)
-		(property "Reference" "H3"
-			(at 232.41 359.4099 0)
-			(show_name no)
-			(do_not_autoplace no)
-			(effects
-				(font
-					(size 1.27 1.27)
-				)
-				(justify left)
-			)
-		)
-		(property "Value" "MountingHole"
-			(at 232.41 361.9499 0)
-			(show_name no)
-			(do_not_autoplace no)
-			(effects
-				(font
-					(size 1.27 1.27)
-				)
-				(justify left)
-			)
-		)
-		(property "Footprint" "MountingHole:MountingHole_3.2mm_M3"
-			(at 229.87 360.68 0)
-			(hide yes)
-			(show_name no)
-			(do_not_autoplace no)
-			(effects
-				(font
-					(size 1.27 1.27)
-				)
-			)
-		)
-		(property "Datasheet" ""
-			(at 229.87 360.68 0)
-			(hide yes)
-			(show_name no)
-			(do_not_autoplace no)
-			(effects
-				(font
-					(size 1.27 1.27)
-				)
-			)
-		)
-		(property "Description" "Mounting Hole without connection"
-			(at 229.87 360.68 0)
-			(hide yes)
-			(show_name no)
-			(do_not_autoplace no)
-			(effects
-				(font
-					(size 1.27 1.27)
-				)
-			)
-		)
-		(instances
-			(project "frambu-v-0-rev-a"
-				(path "/abe203a7-9d57-48b6-8b01-f2c6245f8096"
-					(reference "H3")
-					(unit 1)
-				)
-			)
-		)
-	)
-	(symbol
 		(lib_id "power:GND")
 		(at 167.005 241.935 0)
@@
 					(unit 1)
 				)
+			)
+		)
+	)
+	(symbol
+		(lib_id "Audio:SGTL5000XNLA3")
+		(at 232.41 182.88 0)
+		(unit 1)
+		(body_style 1)
+		(exclude_from_sim no)
+		(in_bom yes)
+		(on_board yes)
+		(in_pos_files yes)
+		(dnp no)
+		(fields_autoplaced yes)
+		(property "Reference" "U4"
+			(at 234.5533 210.82 0)
+			(show_name no)
+			(do_not_autoplace no)
+			(effects
+				(font
+					(size 1.27 1.27)
+				)
+				(justify left)
+			)
+		)
+		(property "Value" "SGTL5000XNLA3"
+			(at 234.5533 213.36 0)
+			(show_name no)
+			(do_not_autoplace no)
+			(effects
+				(font
+					(size 1.27 1.27)
+				)
+				(justify left)
+			)
+		)
+		(property "Footprint" "Package_DFN_QFN:QFN-20-1EP_3x3mm_P0.4mm_EP1.65x1.65mm"
+			(at 232.41 182.88 0)
+			(hide yes)
+			(show_name no)
+			(do_not_autoplace no)
+			(effects
+				(font
+					(size 1.27 1.27)
+				)
+			)
+		)
+		(property "Datasheet" "https://www.nxp.com/docs/en/data-sheet/SGTL5000.pdf"
+			(at 232.41 182.88 0)
+			(hide yes)
+			(show_name no)
+			(do_not_autoplace no)
+			(effects
+				(font
+					(size 1.27 1.27)
+				)
+			)
+		)
+		(property "Description" "Low Power Stereo Codec with Headphone Amp, QFN-20"
+			(at 232.41 182.88 0)
+			(hide yes)
+			(show_name no)
+			(do_not_autoplace no)
+			(effects
+				(font
+					(size 1.27 1.27)
+				)
+			)
+		)
+		(pin "16"
+		)
+		(pin "15"
+		)
+		(pin "3"
+		)
+		(pin "5"
+		)
+		(pin "7"
+		)
+		(pin "6"
+		)
+		(pin "4"
+		)
+		(pin "8"
+		)
+		(pin "1"
+		)
+		(pin "2"
+		)
+		(pin "14"
+		)
+		(pin "9"
+		)
+		(pin "10"
+		)
+		(pin "12"
+		)
+		(pin "11"
+		)
+		(pin "13"
+		)
+		(pin "20"
+		)
+		(pin "19"
+		)
+		(pin "17"
+		)
+		(pin "21"
+		)
+		(pin "18"
+		)
+		(instances
+			(project "frambu-v-0-rev-a"
+				(path "/abe203a7-9d57-48b6-8b01-f2c6245f8096"
+					(reference "U4")
+					(unit 1)
+				)

Commit message: agregar version de pcb
Parts:
- removed C12, C18: 100u, frambu-v-0-rev-a:C1206, symbol Device:C
- removed C15: 10u, Capacitor_SMD:CP_Elec_4x5.4, symbol Device:C
- removed H1, H2: MountingHole, MountingHole:MountingHole_3.2mm_M3, symbol Mechanical:MountingHole
- removed J3, J4: Conn_02x18_Odd_Even, Connector_PinSocket_2.54mm:PinSocket_1x20_P2.54mm_Vertical, symbol Connector_Generic:Conn_02x18_Odd_Even
- removed U2: AMS1117-5.0, Package_TO_SOT_SMD:SOT-223-3_TabPin2, symbol Regulator_Linear:AMS1117-5.0
- removed U4: SGTL5000XNLA3, Package_DFN_QFN:QFN-20-1EP_3x3mm_P0.4mm_EP1.65x1.65mm, symbol Audio:SGTL5000XNLA3
- added J2: pico_pines_1-20, Connector_PinSocket_2.54mm:PinSocket_1x20_P2.54mm_Vertical, symbol Connector_Generic:Conn_01x20
- added J3: SWD, Connector_PinHeader_2.54mm:PinHeader_1x03_P2.54mm_Vertical, symbol Connector_Generic:Conn_01x03
- added J4: GPIO_extra, Connector_PinSocket_2.54mm:PinSocket_1x04_P2.54mm_Vertical, symbol Connector_Generic:Conn_01x04
- added J5: pico_pines_40-21, Connector_PinSocket_2.54mm:PinSocket_1x20_P2.54mm_Vertical, symbol Connector_Generic:Conn_01x20
- added U3: AMS1117-3.3, frambu-v-0-rev-a:SOT-89-3_L4.5-W2.5-P1.50-LS4.2-BR, symbol Regulator_Linear:AMS1117-3.3
- C1: renamed from C16; footprint (none) -> frambu-v-0-rev-a:C0402; LCSC (none) -> C1548
- C10, C7, C8: footprint Capacitor_SMD:C_0805_2012Metric -> frambu-v-0-rev-a:C0402; LCSC (none) -> C307331
- C11: renamed from C3; footprint Capacitor_SMD:C_0805_2012Metric -> frambu-v-0-rev-a:C0402; LCSC (none) -> C307331
- C12: renamed from C11; footprint Capacitor_SMD:C_0805_2012Metric -> frambu-v-0-rev-a:C0402; LCSC (none) -> C307331
- C13: renamed from C4; footprint Capacitor_SMD:C_0805_2012Metric -> frambu-v-0-rev-a:C0402; LCSC (none) -> C307331
- C14: renamed from C9; LCSC (none) -> C77083
- C16: renamed from C5; footprint Capacitor_SMD:C_0805_2012Metric -> frambu-v-0-rev-a:C0402; LCSC (none) -> C307331
- C2: renamed from C17; footprint (none) -> frambu-v-0-rev-a:C0402; LCSC (none) -> C1548
- C4: renamed from C6; footprint Capacitor_SMD:C_0805_2012Metric -> frambu-v-0-rev-a:C0402; LCSC (none) -> C307331
- C5: renamed from C1; LCSC (none) -> C77083
- C9: renamed from C2; footprint Capacitor_SMD:C_0805_2012Metric -> frambu-v-0-rev-a:C0402; LCSC (none) -> C307331
- J1: renamed from J5; footprint frambu-v-0-rev-a:USB-C_SMD-TYPE-C-31-M-12_1 -> Connector_USB:USB_C_Receptacle_HRO_TYPE-C-31-M-12
- R1: renamed from R3; LCSC C11702 -> C2907232
- R5: value 1K -> 1k; LCSC (none) -> C2907232
- R6: renamed from R1; value 27.4 -> 27; footprint (none) -> frambu-v-0-rev-a:R0402; LCSC (none) -> C25100
- R7: renamed from R2; value 27.4 -> 27; footprint (none) -> frambu-v-0-rev-a:R0402; LCSC (none) -> C25100
- U2: renamed from U1; LCSC (none) -> C2040
- Y1: value Crystal_GND24 -> 12MHz; footprint (none) -> Crystal:Crystal_SMD_3225-4Pin_3.2x2.5mm; LCSC (none) -> C20625731
- renumbered C19 to C15, C20 to C3, C13 to C6, R4 to R2, R7 to R3, R6 to R4, U3 to U1
Connections:
- net +3.3V is gone; now on net +3V3: C15.1
- net NOT_QSPI_SS is gone; now on net QSPI_SS: U2.56 (~{QSPI_SS})
- net USB_D_MINUS is gone; now on net USB_D-: R6.1
- net USB_D_PLUS is gone; now on net USB_D+: R7.1
- net VHI is gone; now on net VBUS: C6.1
- net +3V3: now also J5.5 (Pin_5), J5.6 (Pin_6), U3.2 (VO)
- net GND: now also J2.13 (Pin_13), J2.18 (Pin_18), J2.3 (Pin_3), J2.8 (Pin_8), J3.2 (Pin_2), J5.13 (Pin_13), J5.18 (Pin_18), J5.3 (Pin_3), J5.8 (Pin_8), U3.1 (GND)
- net GPIO00: now also J2.1 (Pin_1)
- net GPIO01: now also J2.2 (Pin_2)
- net GPIO02: now also J2.4 (Pin_4)
- net GPIO03: now also J2.5 (Pin_5)
- net GPIO04: now also J2.6 (Pin_6)
- net GPIO05: now also J2.7 (Pin_7)
- net GPIO06: now also J2.9 (Pin_9)
- net GPIO07: now also J2.10 (Pin_10)
- net GPIO08: now also J2.11 (Pin_11)
- net GPIO09: now also J2.12 (Pin_12)
- net GPIO10: now also J2.14 (Pin_14)
- net GPIO11: now also J2.15 (Pin_15)
- net GPIO12: now also J2.16 (Pin_16)
- net GPIO13: now also J2.17 (Pin_17)
- net GPIO14: now also J2.19 (Pin_19)
- net GPIO15: now also J2.20 (Pin_20)
- net GPIO16: now also J5.20 (Pin_20)
- net GPIO17: now also J5.19 (Pin_19)
- net GPIO18: now also J5.17 (Pin_17)
- net GPIO19: now also J5.16 (Pin_16)
- net GPIO20: now also J5.15 (Pin_15)
- net GPIO21: now also J5.14 (Pin_14)
- net GPIO22: now also J5.12 (Pin_12)
- net GPIO23: now also J4.1 (Pin_1)
- net GPIO24: now also J4.2 (Pin_2)
- net GPIO25: now also J4.3 (Pin_3)
- net GPIO26_ADC0: now also J5.10 (Pin_10)
- net GPIO27_ADC1: now also J5.9 (Pin_9)
- net GPIO28_ADC2: now also J5.7 (Pin_7)
- net GPIO29_ADC3: now also J4.4 (Pin_4)
- net RUN: now also J5.11 (Pin_11)
- net SWCLK: now also J3.1 (Pin_1)
- net SWD: now also J3.3 (Pin_3)
- net VBUS: now also J5.1 (Pin_1), U3.3 (VI)
- no-connect marks 2 -> 4
Other:
- title: frambu -> frambu-rev-0
- moved on the sheet: R3

Commit message: agregar mas componentes
Other:
- note removed: "cristal TODO"
Changed lines of the file:
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@@
-		)
-	)
-	(text "cristal TODO\n\n "
-		(exclude_from_sim no)
-		(at 41.275 350.52 0)
-		(effects
-			(font
-				(size 1.27 1.27)
-			)
 		)
 	)

Commit message: agregar nueva version frambu
Parts:
- removed J4: GPIO_extra, Connector_PinSocket_2.54mm:PinSocket_1x04_P2.54mm_Vertical, symbol Connector_Generic:Conn_01x04
Other:
- moved on the sheet: U3
